File: pin-gm-kicad/pin-gm-kicad.kicad_sch (KiCad schematic)
At the start: 40 parts, among them U1 LM358, U2 TL072

Commit message: mostmár tuti jó a layout
Parts:
- BT1: value Battery -> (none); footprint Homemade:SolderWire-homemade -> (none)
- C1, C10, C11, C14, C2, C6, C9: value 100n -> (none); footprint Homemade:C_1206_3216Metric_homemade -> (none)
- C12, C15: value 47u -> (none); footprint Homemade:C_1210_3225Metric_homemade -> (none)
- C13, C3, C5, C7, C8: value 10p -> (none); footprint Homemade:C_1206_3216Metric_homemade -> (none)
- C4: value 10-40p -> (none); footprint Homemade:C_trimmer_D10mm_homemade -> (none)
- D1, D2, D3, D4: value BPW34 -> (none); footprint Homemade:BPW34_homemade -> (none)
- H2: value MountingHole_Pad -> (none); footprint Homemade:Mounting_Hole_Dhole4mm_homemade -> (none)
- L1: value 1m -> (none); footprint Homemade:L_Bourns_SRR0604_homemade -> (none)
- LS1: value Speaker -> (none); footprint Homemade:SolderWire-homemade -> (none)
- R1, R10, R4, R7, R9: value 1k -> (none); footprint Homemade:R_1206_3216Metric_homemade -> (none)
- R11, R12: value 10k -> (none); footprint Homemade:R_1206_3216Metric_homemade -> (none)
- R13: value 100k -> (none); footprint Homemade:R_1206_3216Metric_homemade -> (none)
- R2, R3: value 5k1 -> (none); footprint Homemade:R_1206_3216Metric_homemade -> (none)
- R5: value 4.7k -> (none); footprint Homemade:R_1206_3216Metric_homemade -> (none)
- R6: value 15k -> (none); footprint Homemade:R_1206_3216Metric_homemade -> (none)
- R8: value 10M -> (none); footprint Homemade:R_1206_3216Metric_homemade -> (none)
- RV1: value 5k -> (none); footprint Homemade:Potentiometer_D10_vert_homemade -> (none)
- U1: value LM358 -> (none); footprint Homemade:SO-8_3.9x4.9mm_homemade -> (none)
- U2: value TL072 -> (none); footprint Homemade:SO-8_3.9x4.9mm_homemade -> (none)
